File: hardware/ai_mobile_reader_routed.kicad_pcb (KiCad board)
At the start: 4 copper layers, 58 x 102 mm, 72 parts, among them J1 USB-C, J2 1S_PROTECTED_LIPO, J3 OSPTEK_4.26IN_24PIN, J4 SD_MODULE_2X8, J5 EXTERNAL_KEYS, Q1 AO3400A 30V, SW1 RESET, SW2 BOOT, U1 ESP32-S3-WROOM-1-N16R8, U2 BQ24074RGT, U3 TPS63031DSK

Commit message: feat: 优化pcb
Parts:
- added C25: 100nF, C_0603_1608Metric, F.Cu at (41.0, 47.0)
- added C26: 10uF/6.3V, C_0805_2012Metric, F.Cu at (41.0, 50.0)
- added R21: 10k, R_0603_1608Metric, F.Cu at (41.0, 53.0)
- added R22: 10k, R_0603_1608Metric, F.Cu at (41.0, 56.0)
- added R23: 10k, R_0603_1608Metric, F.Cu at (41.0, 59.0)
- added R24: 47k, R_0603_1608Metric, F.Cu at (47.0, 60.0)
- added R25: 47k, R_0603_1608Metric, F.Cu at (52.0, 60.0)
- J4: value SD_MODULE_2X8 -> Molex 104031-0811 MicroSD; footprint PinHeader_2x08_P2.54mm_Vertical -> microSD_HC_Molex_104031-0811
- moved TP8 18.1 mm to (54.0, 73.0)
- moved TP7 18.0 mm to (47.0, 73.0)
- moved J4 12.7 mm to (52.0, 51.0)
- moved TP6 2.00 mm to (37.5, 55.0)
Connections:
- J4 pad 1: GND -> SD_DAT2
- J4 pad 10: SPI_SCK -> (no net)
- J4 pad 2: GND -> SD_CS
- J4 pad 3: +3V3 -> SPI_MOSI
- J4 pad 5: SD_CS -> SPI_SCK
- J4 pad 6: SD_CS -> GND
- J4 pad 7: SPI_MOSI -> SD_MISO
- J4 pad 8: SPI_MOSI -> SD_DAT1
- J4 pad 9: SPI_SCK -> (no net)
Routing:
- net GND: track 520.1 -> 115.7 mm, vias 3 -> 52
- net +3V3: track 195.4 -> 219.4 mm, vias 6 -> 2
- net SD_DAT1: track 0.00 -> 15.5 mm, vias 0 -> 2
- net EPD_BUSY: track 52.6 -> 67.4 mm
- net BTN_HOME: track 31.8 -> 43.8 mm
- net USB_VBUS: track 59.1 -> 69.7 mm, vias 5 -> 4
- net SD_CS: track 22.6 -> 32.8 mm, vias 1 -> 2
- net SD_DAT2: track 0.00 -> 8.99 mm
- net BTN_DOWN: track 29.2 -> 37.4 mm, vias 2 -> 1
- net SD_MISO: track 27.7 -> 35.8 mm, vias 1 -> 0
- net SPI_SCK: track 67.5 -> 60.1 mm, vias 2 -> 3
- net PREVGH: track 49.1 -> 41.9 mm
- net EPD_CS: track 60.3 -> 53.1 mm
- net BAT_ADC: track 74.5 -> 79.9 mm, vias 2 -> 3
- net EPD_GDR: track 34.8 -> 39.6 mm, vias 2 -> 1
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